File: Circuit/Hapticreactor_Driver/DAC.kicad_sch (KiCad schematic)
At the start: 4 parts, among them U3 MCP4725xxx-xCH

Commit message: ハプティックリアクタ用基板完成
Parts:
- C5: value C -> 0.1u
Changed lines of the file:
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@@
 			)
 		)
-		(property "Value" "C"
+		(property "Value" "0.1u"
 			(at 120.65 81.2799 0)
 			(effects

Commit message: VMをバッテリ入力に変更，バッテリ周りの間違いを訂正
Changed lines of the file:
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@@
 	(generator_version "9.0")
 	(paper "A4")
-	(text_box "IIC_Address_Select\nNC:0x60\nConnected:0x61\n"
+	(text_box "IIC_Address_Select\nNC:0x62\nConnected:0x63\n"
 		(exclude_from_sim no)
 		(at 167.132 62.738 0)
@@
 		)
 		(property "Value" "MCP4725xxx-xCH"
-			(at 122.936 76.708 0)
-			(effects
-				(font
+			(at 131.572 76.454 0)
+			(effects
+				(font
